File: megafrank.kicad_pcb (KiCad board)
At the start: 2 copper layers, 149.9 x 99.5 mm, 262 parts, among them J1 UART, J10 RCA-103, J11 Pin Header 1x08, J12 SJ1-3525N, J13 PAM L, J14 PAM R, J15 SJ1-3525N, J16 GP2, J17 GP2, J18 104031-0811, J19 SS-52100-004, J2 DEBUG, J20 VGA, J21 SS-52100-004, J3 PWR, J4 Conn_02x20_Odd_Even, J5 DC-005-5A-2.0, J6 USB4215-03-A, J7 MDC-036, J8 BAT 3V, J9 DC3RX19JA2, Q1 BC850, U1 MP1584EN-LF-Z, U10 DS3231MZ, U11 DS2401P+, U12 ESP-PSRAM64, U13 MW7211A, U14 Pimoroni PGA2350, U15 74HC4052D, U16 ESP-01v090, U17 CD4069UBM, U18 TDA1387T, U19 PAM8403D, U2 USBLC6-2SC6, U20 LM358, U21 74HC4052D, U3 AMS1117 3.3, U4 TXS0104EDR, U5 JFC95101, U6 74HC74, U7 JFC95101, U8 74HC595, U9 74HC595, X1 3.58 MHz

Commit message: update silkscreen and vias
Routing:
- net Net-(H5-+): track 60.2 -> 42.2 mm, vias 4 -> 2
- net /Audio/TS/R_IN: track 123.9 -> 116.4 mm
- net /Audio/TS/BEEP: track 39.3 -> 36.8 mm, vias 3 -> 2
- net /PGPIO31: track 33.7 -> 32.5 mm
- net /Audio/TS/YM_CS1: track 37.1 -> 38.3 mm
- net +3V3: track 412.5 -> 411.7 mm
- net GND: vias 219 -> 245
Other:
- board text added: "2 1"
- board text added: "40 39"
- board text added: "Designed by Mikhail Matveev https://frank.rh1.tech U4 updated by Eugene Stahov @ub8cjz https://github.com/evgs/mega-frank-u4"
- board text added: "GP0/TX GND GP1/RX"
- board text added: "OFF ON"
- board text added: "SWDIO GND SWCLK"
- board text added: "TYPE-C HUB"
- board text removed: "Designed by Mikhail Matveev https://frank.rh1.tech U4 updated by Eugene Stahov https://github.com/evgs/mega-frank-u4"
